Commit message: Add files via upload

File: 1.urdf (robot description, URDF)
Before this commit: robot robots/1, 6 links, 5 joints
Links:
- link 1844789: mass 0.025620554769945746 -> 0.022543488066187885; geometry collision cylinder length=0.09698090677467489 radius=0.009928035035897387
- link 3416624: mass 0.29737445246817784 -> 0.8541329457565685; geometry collision capsule length=0.04143685882263688 radius=0.05818503294385344
- link 4064029: mass 0.4940959173612819 -> 0.32657421908334666; geometry collision cylinder length=0.09571551589530464 radius=0.0368241539840548
Joints:
- joint 2951283: limit lower=0 upper=6.283185307179586 effort=1 velocity=1 -> lower=0 upper=0 effort=1 velocity=1; type revolute -> continuous
- joint 3283812: limit lower=0 upper=6.283185307179586 effort=1 velocity=1 -> lower=0 upper=0 effort=1 velocity=1; type revolute -> continuous

File: 2.urdf (robot description, URDF)
Before this commit: robot robots/2, 6 links, 5 joints
Links:
- removed link 7664932
- added link 7526257, mass 0.0174644118202432; collision sphere radius=0.06747523222590207
- link 1917999: mass 1.0319173404817041 -> 1.6992584420914167; geometry collision sphere radius=0.07506861412184562
- link 4668302: mass 2.1220262946419868 -> 1.9117785545564248; geometry collision sphere radius=0.09571551589530464
- link 9160297: mass 0.22011334635223626 -> 0.018000647853530338; geometry collision cylinder length=0.0018789800436355142 radius=0.05684339488686485
Joints:
- removed joint 341845
- removed joint 6687090
- added joint 4219081: type continuous, parent 1917999, child 7526257, origin xyz=0.00300498 0.07421909 0.06421532 rpy=-1.7160003618167112 0.040040437173014407 -0.04631943652625425, axis 0 0 1, limit lower=0 upper=0 effort=1 velocity=1
- added joint 4295565: type fixed, parent 9160297, child 1917999, origin xyz=3.50301186e-02 6.44194645e-02 4.28995226e-18 rpy=0 3.141592653589793 0, axis 0 0 0, limit lower=0 upper=0 effort=10 velocity=10
- joint 2527987: limit lower=0 upper=0 effort=1 velocity=1 -> lower=0 upper=6.283185307179586 effort=1 velocity=1; type continuous -> revolute
- joint 7329820: origin xyz= 0.00322155 -0.01019242  0.01820433 rpy=-0.0 1.5707963267948963 0.0 -> xyz= 0.00053562 -0.01258534  0.03843817 rpy=0 0 0
- joint 86107: axis 0 0 1 -> 0 0 0; limit lower=0 upper=6.283185307179586 effort=1 velocity=1 -> lower=0 upper=0 effort=10 velocity=10; origin xyz= 0.06016102 -0.01880747  0.16778593 rpy=0.24650908055781443 0.7035514966856717 0.09087760815071198 -> xyz=0.08061522 0.03688976 0.13179586 rpy=-0.7964900551149955 1.0014207784228513 -0.4525773058843282; type revolute -> fixed
